File: layout_kicad/esp01carrier.kicad_pcb (KiCad board)
At the start: 2 copper layers, 49.5 x 35.6 mm, 18 parts, among them J1 ESP-01, J2 REED1, J3 REED2, J4 Vin 5V, U1 CD74HCT86E, U2 SN74HCT32N, U3 HT7333

Commit message: Change RC-curcuits to reduce current
Parts:
- removed REF**: MountingHole_3mm, Mounting_Holes:MountingHole_3mm
- C1, C2: value 100uF -> 10uF
- J1: footprint Pin_Headers:Pin_Header_Straight_2x04_Pitch2.54mm -> Socket_Strips:Socket_Strip_Straight_2x04_Pitch2.54mm
- R1, R2, R4, R5: value 10k -> 100k
Changed lines of the file:
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@@
     (tracks 103)
     (zones 0)
-    (modules 18)
+    (modules 17)
     (nets 17)
   )
@@
     (add_net RST)
     (add_net RX)
+  )
+  (module Socket_Strips:Socket_Strip_Straight_2x04_Pitch2.54mm (layer F.Cu)
+    (at 137.795 123.19)
+    (descr "Through hole straight socket strip, 2x04, 2.54mm pitch, double rows")
+    (tags "Through hole socket strip THT 2x04 2.54mm double row")
+    (fp_text reference J1 (at -1.27 -2.33) (layer F.SilkS)
+      (effects (font (size 1 1) (thickness 0.15)))
+    )
+    (fp_text value ESP-01 (at -1.27 9.95) (layer F.Fab)
+      (effects (font (size 1 1) (thickness 0.15)))
+    )
+    (fp_text user %R (at -1.27 -2.33) (layer F.Fab)
+      (effects (font (size 1 1) (thickness 0.15)))
+    )
+    (fp_line (start 1.8 -1.8) (end -4.35 -1.8) (layer F.CrtYd) (width 0.05))
+    (fp_line (start 1.8 9.4) (end 1.8 -1.8) (layer F.CrtYd) (width 0.05))
+    (fp_line (start -4.35 9.4) (end 1.8 9.4) (layer F.CrtYd) (width 0.05))
+    (fp_line (start -4.35 -1.8) (end -4.35 9.4) (layer F.CrtYd) (width 0.05))
+    (fp_line (start 1.33 -1.33) (end 0.06 -1.33) (layer F.SilkS) (width 0.12))
+    (fp_line (start 1.33 0) (end 1.33 -1.33) (layer F.SilkS) (width 0.12))
+    (fp_line (start -1.27 1.27) (end 1.33 1.27) (layer F.SilkS) (width 0.12))
+    (fp_line (start -1.27 -1.33) (end -1.27 1.27) (layer F.SilkS) (width 0.12))
+    (fp_line (start -3.87 -1.33) (end -1.27 -1.33) (layer F.SilkS) (width 0.12))
+    (fp_line (start -3.87 8.95) (end -3.87 -1.33) (layer F.SilkS) (width 0.12))
+    (fp_line (start 1.33 8.95) (end -3.87 8.95) (layer F.SilkS) (width 0.12))
+    (fp_line (start 1.33 1.27) (end 1.33 8.95) (layer F.SilkS) (width 0.12))
+    (fp_line (start 1.27 -1.27) (end -3.81 -1.27) (layer F.Fab) (width 0.1))
+    (fp_line (start 1.27 8.89) (end 1.27 -1.27) (layer F.Fab) (width 0.1))
+    (fp_line (start -3.81 8.89) (end 1.27 8.89) (layer F.Fab) (width 0.1))
+    (fp_line (start -3.81 -1.27) (end -3.81 8.89) (layer F.Fab) (width 0.1))
+    (pad 8 thru_hole oval (at -2.54 7.62) (size 1.7 1.7) (drill 1) (layers *.Cu *.Mask)
+      (net 16 RX))
+    (pad 7 thru_hole oval (at 0 7.62) (size 1.7 1.7) (drill 1) (layers *.Cu *.Mask)
+      (net 5 +3V3))
+    (pad 6 thru_hole oval (at -2.54 5.08) (size 1.7 1.7) (drill 1) (layers *.Cu *.Mask)
+      (net 7 GPIO0))
+    (pad 5 thru_hole oval (at 0 5.08) (size 1.7 1.7) (drill 1) (layers *.Cu *.Mask)
+      (net 6 RST))
+    (pad 4 thru_hole oval (at -2.54 2.54) (size 1.7 1.7) (drill 1) (layers *.Cu *.Mask)
+      (net 15 "Net-(J1-Pad4)"))
+    (pad 3 thru_hole oval (at 0 2.54) (size 1.7 1.7) (drill 1) (layers *.Cu *.Mask)
+      (net 5 +3V3))
+    (pad 2 thru_hole oval (at -2.54 0) (size 1.7 1.7) (drill 1) (layers *.Cu *.Mask)
+      (net 3 GND))
+    (pad 1 thru_hole rect (at 0 0) (size 1.7 1.7) (drill 1) (layers *.Cu *.Mask)
+      (net 4 "Net-(J1-Pad1)"))
+    (model ${KISYS3DMOD}/Socket_Strips.3dshapes/Socket_Strip_Straight_2x04_Pitch2.54mm.wrl
+      (offset (xyz -1.269999980926514 -3.809999942779541 0))
+      (scale (xyz 1 1 1))
+      (rotate (xyz 0 0 270))
+    )
   )
   (module Capacitors_THT:CP_Radial_D5.0mm_P2.50mm (layer F.Cu)
@@
       (effects (font (size 1 1) (thickness 0.15)))
     )
-    (fp_text value 10k (at 3.81 2.31 90) (layer F.Fab)
+    (fp_text value 100k (at 3.81 2.31 90) (layer F.Fab)
       (effects (font (size 1 1) (thickness 0.15)))
     )
@@
       (effects (font (size 1 1) (thickness 0.15)))
     )
-    (fp_text value 10k (at 9.525 4.445 180) (layer F.Fab)
+    (fp_text value 100k (at 9.525 4.445 180) (layer F.Fab)
       (effects (font (size 1 1) (thickness 0.15)))
     )
@@
       (scale (xyz 1 1 1))
       (rotate (xyz 0 0 0))
-    )
-  )
-  (module Pin_Headers:Pin_Header_Straight_2x04_Pitch2.54mm (layer F.Cu)
-    (at 137.795 123.19)
-    (descr "Through hole straight pin header, 2x04, 2.54mm pitch, double rows")
-    (tags "Through hole pin header THT 2x04 2.54mm double row")
-    (fp_text reference J1 (at 1.27 -2.33) (layer F.SilkS) hide
-      (effects (font (size 1 1) (thickness 0.15)))
-    )
-    (fp_text value ESP-01 (at 1.27 9.95) (layer F.Fab)
-      (effects (font (size 1 1) (thickness 0.15)))
-    )
-    (fp_line (start 0 -1.27) (end 3.81 -1.27) (layer F.Fab) (width 0.1))
-    (fp_line (start 3.81 -1.27) (end 3.81 8.89) (layer F.Fab) (width 0.1))
-    (fp_line (start 3.81 8.89) (end -1.27 8.89) (layer F.Fab) (width 0.1))
-    (fp_line (start -1.27 8.89) (end -1.27 0) (layer F.Fab) (width 0.1))
-    (fp_line (start -1.27 0) (end 0 -1.27) (layer F.Fab) (width 0.1))
-    (fp_line (start -1.33 8.95) (end 3.87 8.95) (layer F.SilkS) (width 0.12))
-    (fp_line (start -1.33 1.27) (end -1.33 8.95) (layer F.SilkS) (width 0.12))
-    (fp_line (start 3.87 -1.33) (end 3.87 8.95) (layer F.SilkS) (width 0.12))
-    (fp_line (start -1.33 1.27) (end 1.27 1.27) (layer F.SilkS) (width 0.12))
-    (fp_line (start 1.27 1.27) (end 1.27 -1.33) (layer F.SilkS) (width 0.12))
-    (fp_line (start 1.27 -1.33) (end 3.87 -1.33) (layer F.SilkS) (width 0.12))
-    (fp_line (start -1.33 0) (end -1.33 -1.33) (layer F.SilkS) (width 0.12))
-    (fp_line (start -1.33 -1.33) (end 0 -1.33) (layer F.SilkS) (width 0.12))
-    (fp_line (start -1.8 -1.8) (end -1.8 9.4) (layer F.CrtYd) (width 0.05))
-    (fp_line (start -1.8 9.4) (end 4.35 9.4) (layer F.CrtYd) (width 0.05))
-    (fp_line (start 4.35 9.4) (end 4.35 -1.8) (layer F.CrtYd) (width 0.05))
-    (fp_line (start 4.35 -1.8) (end -1.8 -1.8) (layer F.CrtYd) (width 0.05))
-    (fp_text user %R (at 1.27 3.81 90) (layer F.Fab) hide
-      (effects (font (size 1 1) (thickness 0.15)))
-    )
-    (pad 1 thru_hole rect (at 0 0) (size 1.7 1.7) (drill 1) (layers *.Cu *.Mask)
-      (net 4 "Net-(J1-Pad1)"))
-    (pad 2 thru_hole oval (at 2.54 0) (size 1.7 1.7) (drill 1) (layers *.Cu *.Mask)
-      (net 3 GND))
-    (pad 3 thru_hole oval (at 0 2.54) (size 1.7 1.7) (drill 1) (layers *.Cu *.Mask)
-      (net 5 +3V3))
-    (pad 4 thru_hole oval (at 2.54 2.54) (size 1.7 1.7) (drill 1) (layers *.Cu *.Mask)
-      (net 15 "Net-(J1-Pad4)"))
-    (pad 5 thru_hole oval (at 0 5.08) (size 1.7 1.7) (drill 1) (layers *.Cu *.Mask)
-      (net 6 RST))
-    (pad 6 thru_hole oval (at 2.54 5.08) (size 1.7 1.7) (drill 1) (layers *.Cu *.Mask)
-      (net 7 GPIO0))
-    (pad 7 thru_hole oval (at 0 7.62) (size 1.7 1.7) (drill 1) (layers *.Cu *.Mask)
-      (net 5 +3V3))
-    (pad 8 thru_hole oval (at 2.54 7.62) (size 1.7 1.7) (drill 1) (layers *.Cu *.Mask)
-      (net 16 RX))
-    (model ${KISYS3DMOD}/Socket_Strips.3dshapes/Socket_Strip_Straight_2x04_Pitch2.54mm.wrl
-      (offset (xyz 1.27 -3.81 0))
-      (scale (xyz 1 1 1))
-      (rotate (xyz 0 0 90))
-    )
-    (model C:/Users/joachim/workspace/tor/esp01/esp01.wrl
-      (offset (xyz 0 -3.81 11))
-      (scale (xyz 0.39 0.39 0.39))
-      (rotate (xyz 0 180 -180))
     )
   )
@@
       (effects (font (size 1 1) (thickness 0.15)))
     )
-    (fp_text value 100uF (at 1.25 5.06 90) (layer F.Fab)
+    (fp_text value 10uF (at 1.25 5.06 90) (layer F.Fab)
       (effects (font (size 1 1) (thickness 0.15)))
     )
@@
       (effects (font (size 1 1) (thickness 0.15)))
     )
-    (fp_text value 100uF (at 1.27 4.445 90) (layer F.Fab)
+    (fp_text value 10uF (at 1.27 4.445 90) (layer F.Fab)
       (effects (font (size 1 1) (thickness 0.15)))
     )
@@
       (effects (font (size 1 1) (thickness 0.15)))
     )
-    (fp_text value 10k (at 3.81 5.08) (layer F.Fab)
+    (fp_text value 100k (at 3.81 5.08) (layer F.Fab)
       (effects (font (size 1 1) (thickness 0.15)))
     )
@@
       (effects (font (size 1 1) (thickness 0.15)))
     )
-    (fp_text value 10k (at 6.985 -2.54) (layer F.Fab)
+    (fp_text value 100k (at 6.985 -2.54) (layer F.Fab)
       (effects (font (size 1 1) (thickness 0.15)))
     )
@@
     )
   )
-  (module Mounting_Holes:MountingHole_3mm (layer F.Cu)
-    (at 138.43 104.775)
-    (descr "Mounting Hole 3mm, no annular")
-    (tags "mounting hole 3mm no annular")
-    (attr virtual)
-    (fp_text reference REF** (at 0 -4) (layer F.SilkS) hide
-      (effects (font (size 1 1) (thickness 0.15)))
-    )
-    (fp_text value MountingHole_3mm (at 0 4) (layer F.Fab) hide
-      (effects (font (size 1 1) (thickness 0.15)))
-    )
-    (fp_text user %R (at 0.3 0) (layer F.Fab)
-      (effects (font (size 1 1) (thickness 0.15)))
-    )
-    (fp_circle (center 0 0) (end 3 0) (layer Cmts.User) (width 0.15))
-    (fp_circle (center 0 0) (end 3.25 0) (layer F.CrtYd) (width 0.05))
-    (pad 1 np_thru_hole circle (at 0 0) (size 3 3) (drill 3) (layers *.Cu *.Mask))
-  )
   (module Capacitors_THT:CP_Radial_D6.3mm_P2.50mm (layer F.Cu)
